File: PCB/key-shift-pcb.kicad_sch (KiCad schematic)
At the start: 0 parts

Commit message: adding matrix schematic
Parts:
- added D1, D10, D11, D12, D13, D14, D15, D16, D2, D3, D4, D5, D6, D7, D8, D9: D, symbol Device:D
- added SW1, SW10, SW11, SW12, SW13, SW14, SW15, SW16, SW2, SW3, SW4, SW5, SW6, SW7, SW8, SW9: SW_SPST, symbol Switch:SW_SPST
- added U1: STM32F411CEUx, Package_DFN_QFN:QFN-48-1EP_7x7mm_P0.5mm_EP5.6x5.6mm, symbol MCU_ST_STM32F4:STM32F411CEUx
Connections:
- new net: D2.2 (A), SW2.2 (B)
- new net: D1.2 (A), SW1.2 (B)
- new net: D15.2 (A), SW15.2 (B)
- new net: D16.2 (A), SW16.2 (B)
- new net: D11.2 (A), SW11.2 (B)
- new net: D13.2 (A), SW13.2 (B)
- new net: D3.2 (A), SW3.2 (B)
- new net: U1.23 (VSS), U1.35 (VSS), U1.47 (VSS), U1.49 (VSS)
- new net: D9.2 (A), SW9.2 (B)
- new net: D14.2 (A), SW14.2 (B)
- new net: D7.2 (A), SW7.2 (B)
- new net: D12.2 (A), SW12.2 (B)
- new net: D8.2 (A), SW8.2 (B)
- new net: D4.2 (A), SW4.2 (B)
- new net: D10.2 (A), SW10.2 (B)
- new net: D6.2 (A), SW6.2 (B)
- new net: D5.2 (A), SW5.2 (B)
- new net COLUMN1: SW1.1 (A), SW13.1 (A), SW5.1 (A), SW9.1 (A), U1.14 (PA4)
- new net COLUMN2: SW10.1 (A), SW14.1 (A), SW2.1 (A), SW6.1 (A), U1.15 (PA5)
- new net COLUMN3: SW11.1 (A), SW15.1 (A), SW3.1 (A), SW7.1 (A), U1.16 (PA6)
- new net COLUMN4: SW12.1 (A), SW16.1 (A), SW4.1 (A), SW8.1 (A), U1.17 (PA7)
- new net ROW1: D1.1 (K), D2.1 (K), D3.1 (K), D4.1 (K), U1.10 (PA0)
- new net ROW2: D5.1 (K), D6.1 (K), D7.1 (K), D8.1 (K), U1.11 (PA1)
- new net ROW3: D10.1 (K), D11.1 (K), D12.1 (K), D9.1 (K), U1.12 (PA2)
- new net ROW4: D13.1 (K), D14.1 (K), D15.1 (K), D16.1 (K), U1.13 (PA3)
